File: elkrets/LM386.sch (KiCad schematic (older format))
At the start: 61 parts, among them P1 CONN_2, Q1 PNP, Q2 PNP, Q3 NPN, Q4 NPN, U1 LM386, U2 LM324, U3 4069, U4 74HC377, U5 LM358

Commit message: ELkrets uppdate
Parts:
- removed IN1, Input1, Input2, Input3, Input4, OUT1, Output1, Output2: CONN_1, symbol CONN_1
- added C? (x3): C, ~, symbol C
- added C? (x4): CP1, ~, symbol CP1
- added L?: 10µ, ~, symbol INDUCTOR_SMALL
- added P?: Ultrasonic, symbol CONN_4
- added P?: ICSP, symbol CONN_6
- added P?: Camera, symbol CAMERA
- added P?: Radio, symbol CONN_4X2
- added P? (x2): Motor, symbol CONN_2
- added P?: Jtag, symbol CONN_5X2
- added Q? (x2): PNP, ~, symbol PNP
- added Q? (x2): NPN, ~, symbol NPN
- added R? (x4): 1,5k, ~, symbol R
- added R?: 100R, ~, symbol R
- added R? (x2): 4.7k, ~, symbol R
- added R? (x4): R, ~, symbol R
- added SW? (x2): SW_PUSH, ~, symbol SW_PUSH
- added U?: XC9572XL, ~, symbol XC9572
- P1: value CONN_2 -> Microphone
Connections:
- net labels added: CAMERA_PARALLEL, D0, D1, D2, D3, D4, D5, D6, D7, DAC_SLAVE_SELECT, I2C_BUS, ICSP, ISP, M0, M1, M2, M3, MICROSWITCH, MICRO_L, MICRO_R, MISO, MOSI, MOTOR_GPIO, OE, RADIO_CE, RADIO_CSN, RCK, RRST, RST, RX, SCK, SCL, SDA, SPI BUS, TX, VSYNC, WR, WRST, XC9572_SLAVE_SELECT
- net labels removed: Mic Förstärkare
- wire segments 129 -> 334
- no-connect marks 3 -> 31
Other:
- moved on the sheet: C1, C2, C3, C4, C5, C6, C7, C8, P1, Q1, Q2, Q3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

Commit message: Elkrets labels
Other:
- note added: "Camera"
- note added: "Digital to \nAnalog \nConverter"
- note added: "H-Bridge\n"
- note added: "LPC1114 ARM"
- note added: "Micro-Switches"
- note added: "Microphone"
- note added: "Microphone\nAmplifier"
- note added: "Motors"
- note added: "Ping Sensor"
- note added: "Programming\nHeader"
- note added: "Radio \nLink"
- note added: "Speaker\n"
- note added: "Speaker\nAmplifier"
- note added: "XC9572CPLD"
- moved on the sheet: R?, SW?
Changed lines of the file:
@@
 M3
 Wire Bus Line
-	25550 7600 21950 7600
-Wire Bus Line
-	21950 7600 21950 9450
+	25550 8200 21950 8200
 Wire Bus Line
 	21950 9450 17450 9450
@@
 L SW_PUSH SW?
 U 1 1 536D8AF9
-P 24100 6850
-F 0 "SW?" H 24250 6960 50  0000 C CNN
-F 1 "SW_PUSH" H 24100 6770 50  0000 C CNN
-F 2 "~" H 24100 6850 60  0000 C CNN
-F 3 "~" H 24100 6850 60  0000 C CNN
-	1    24100 6850
+P 24100 7450
+F 0 "SW?" H 24250 7560 50  0000 C CNN
+F 1 "SW_PUSH" H 24100 7370 50  0000 C CNN
+F 2 "~" H 24100 7450 60  0000 C CNN
+F 3 "~" H 24100 7450 60  0000 C CNN
+	1    24100 7450
 	1    0    0    -1
 $EndComp
@@
 L SW_PUSH SW?
 U 1 1 536D8B06
-P 25350 6850
-F 0 "SW?" H 25500 6960 50  0000 C CNN
-F 1 "SW_PUSH" H 25350 6770 50  0000 C CNN
-F 2 "~" H 25350 6850 60  0000 C CNN
-F 3 "~" H 25350 6850 60  0000 C CNN
-	1    25350 6850
-	1    0    0    -1
-$EndComp
-Entry Wire Line
-	23700 7600 23800 7500
-Entry Wire Line
-	24950 7600 25050 7500
-Wire Wire Line
-	25050 6800 25050 7500
-Wire Wire Line
-	23800 6800 23800 7500
+P 25350 7450
+F 0 "SW?" H 25500 7560 50  0000 C CNN
+F 1 "SW_PUSH" H 25350 7370 50  0000 C CNN
+F 2 "~" H 25350 7450 60  0000 C CNN
+F 3 "~" H 25350 7450 60  0000 C CNN
+	1    25350 7450
+	1    0    0    -1
+$EndComp
+Entry Wire Line
+	23700 8200 23800 8100
+Entry Wire Line
+	24950 8200 25050 8100
+Wire Wire Line
+	25050 7400 25050 8100
+Wire Wire Line
+	23800 7400 23800 8100
 $Comp
 L 3V3 #PWR?
 U 1 1 536D8DB0
-P 24500 6150
-F 0 "#PWR?" H 24500 6250 40  0001 C CNN
-F 1 "3V3" H 24500 6275 40  0000 C CNN
-F 2 "" H 24500 6150 60  0000 C CNN
-F 3 "" H 24500 6150 60  0000 C CNN
-	1    24500 6150
+P 24500 6750
+F 0 "#PWR?" H 24500 6850 40  0001 C CNN
+F 1 "3V3" H 24500 6875 40  0000 C CNN
+F 2 "" H 24500 6750 60  0000 C CNN
+F 3 "" H 24500 6750 60  0000 C CNN
+	1    24500 6750
 	1    0    0    -1
 $EndComp
@@
 L R R?
 U 1 1 536D8DBF
-P 23800 6550
-F 0 "R?" V 23880 6550 40  0000 C CNN
-F 1 "4.7k" V 23807 6551 40  0000 C CNN
-F 2 "~" V 23730 6550 30  0000 C CNN
-F 3 "~" H 23800 6550 30  0000 C CNN
-	1    23800 6550
+P 23800 7150
+F 0 "R?" V 23880 7150 40  0000 C CNN
+F 1 "4.7k" V 23807 7151 40  0000 C CNN
+F 2 "~" V 23730 7150 30  0000 C CNN
+F 3 "~" H 23800 7150 30  0000 C CNN
+	1    23800 7150
 	1    0    0    -1
 $EndComp
@@
 L R R?
 U 1 1 536D8DCE
-P 25050 6550
-F 0 "R?" V 25130 6550 40  0000 C CNN
-F 1 "4.7k" V 25057 6551 40  0000 C CNN
-F 2 "~" V 24980 6550 30  0000 C CNN
-F 3 "~" H 25050 6550 30  0000 C CNN
-	1    25050 6550
-	1    0    0    -1
-$EndComp
-Wire Wire Line
-	25050 6300 23800 6300
-Wire Wire Line
-	24500 6150 24500 6300
-Connection ~ 24500 6300
-Connection ~ 23800 6850
-Connection ~ 25050 6850
+P 25050 7150
+F 0 "R?" V 25130 7150 40  0000 C CNN
+F 1 "4.7k" V 25057 7151 40  0000 C CNN
+F 2 "~" V 24980 7150 30  0000 C CNN
+F 3 "~" H 25050 7150 30  0000 C CNN
+	1    25050 7150
+	1    0    0    -1
+$EndComp
+Wire Wire Line
+	25050 6900 23800 6900
+Wire Wire Line
+	24500 6750 24500 6900
+Connection ~ 24500 6900
+Connection ~ 23800 7450
+Connection ~ 25050 7450
 $Comp
 L GND #PWR?
 U 1 1 536D9325
-P 24400 6950
-F 0 "#PWR?" H 24400 6950 30  0001 C CNN
-F 1 "GND" H 24400 6880 30  0001 C CNN
-F 2 "" H 24400 6950 60  0000 C CNN
-F 3 "" H 24400 6950 60  0000 C CNN
-	1    24400 6950
+P 24400 7550
+F 0 "#PWR?" H 24400 7550 30  0001 C CNN
+F 1 "GND" H 24400 7480 30  0001 C CNN
+F 2 "" H 24400 7550 60  0000 C CNN
+F 3 "" H 24400 7550 60  0000 C CNN
+	1    24400 7550
 	1    0    0    -1
 $EndComp
@@
 L GND #PWR?
 U 1 1 536D9332
-P 25650 6950
-F 0 "#PWR?" H 25650 6950 30  0001 C CNN
-F 1 "GND" H 25650 6880 30  0001 C CNN
-F 2 "" H 25650 6950 60  0000 C CNN
-F 3 "" H 25650 6950 60  0000 C CNN
-	1    25650 6950
-	1    0    0    -1
-$EndComp
-Wire Wire Line
-	25650 6850 25650 6950
-Wire Wire Line
-	24400 6850 24400 6950
-Text Label 23800 7450 1    59   ~ 0
+P 25650 7550
+F 0 "#PWR?" H 25650 7550 30  0001 C CNN
+F 1 "GND" H 25650 7480 30  0001 C CNN
+F 2 "" H 25650 7550 60  0000 C CNN
+F 3 "" H 25650 7550 60  0000 C CNN
+	1    25650 7550
+	1    0    0    -1
+$EndComp
+Wire Wire Line
+	25650 7450 25650 7550
+Wire Wire Line
+	24400 7450 24400 7550
+Text Label 23800 8050 1    59   ~ 0
 MICRO_L
-Text Label 25050 7450 1    59   ~ 0
+Text Label 25050 8050 1    59   ~ 0
 MICRO_R
 $Comp
@@
 Wire Wire Line
 	14900 16500 14900 16650
+Text Notes 23450 19150 0    276  ~ 0
+Radio \nLink
+Text Notes 22350 15350 0    276  ~ 0
+Digital to \nAnalog \nConverter
+Text Notes 26350 15250 0    276  ~ 0
+Speaker\nAmplifier
+Text Notes 29450 14950 0    276  ~ 0
+Speaker\n
+Text Notes 13200 19350 0    276  ~ 0
+XC9572CPLD
+Text Notes 7850 18450 0    276  ~ 0
+Camera
+Text Notes 20700 12150 0    276  ~ 0
+Microphone\nAmplifier
+Text Notes 25800 11200 0    276  ~ 0
+Microphone
+Text Notes 22400 8700 0    276  ~ 0
+Micro-Switches
+Wire Bus Line
+	21950 8200 21950 9450
+Text Notes 21200 4150 1    276  ~ 0
+H-Bridge\n
+Text Notes 30350 4250 0    276  ~ 0
+Motors
+Text Notes 16650 4900 0    276  ~ 0
+Ping Sensor
+Text Notes 10800 4950 0    276  ~ 0
+Programming\nHeader
+Text Notes 14200 13250 0    276  ~ 0
+LPC1114 ARM
 $EndSCHEMATC

Commit message: circuit documentation
Parts:
- added SW?: ISP, ~, symbol SW_PUSH
- added SW?: RST, ~, symbol SW_PUSH
- added U?: 8NOR, symbol 8NOR
- added U?: SR8CE, symbol SR8CE
- added U?: DLATCH, symbol DLATCH
- added U?: 2MUX1, symbol 2MUX1
- added U?: SR8CLE, symbol SR8CLE
- added U? (x2): NOT, symbol 74HC04
Connections:
- net labels added: D[0], D[1], D[2], D[3], D[4], D[5], D[6], D[7]
- wire segments 334 -> 381
Other:
- note added: "Camera FIFO reset\n"
- note added: "Internal Logic"
- note added: "Parallel camera data"
- note added: "Parallel data read strobe"
- note added: "Programming mode\nbuttons"
- note added: "Reset state machine\n"
- note added: "Serial command shift in"
- note added: "Serial data shift out"
- note added: "XC9572\nCPLD"
- note removed: "XC9572CPLD"

Commit message: circuit renders
Parts:
- added U? (x2): BUFE, symbol BUFE
Connections:
- net MISO: now also U?.~, U?.~; no longer P?.7
- net RADIO_CSN: now also U?.~
- net XC9572_SLAVE_SELECT: now also U?.~
- net at U?.~: now also U?.~ (Q); no longer U?.~ (SLI)
- new net: P?.7, U?.~
- new net: U?.~, U?.~ (SLI) (x8)
- new net: U?.2, U?.~ (S), U?.~ (SLI), U?.~ (SLI)
- new net: U?.1, U?.~ (Q), U?.~ (S)
Changed lines of the file:
@@
-EESchema Schematic File Version 2  date tis 13 maj 2014 09:56:20
+EESchema Schematic File Version 2  date tis 13 maj 2014 13:19:24
 LIBS:power
 LIBS:device
@@
 encoding utf-8
 Sheet 1 1
-Title ""
+Title "AutoKorg"
 Date "13 may 2014"
 Rev ""
@@
 Comment4 ""
 $EndDescr
-Text Notes 13950 5800 0    90   ~ 0
-Programming mode\nbuttons
+Connection ~ 23200 19450
+Wire Wire Line
+	23200 19450 23000 19450
+Wire Wire Line
+	23000 19450 23000 19700
+Wire Wire Line
+	23100 18650 22700 18650
+Wire Wire Line
+	23100 18650 23100 20100
+Wire Wire Line
+	22800 19550 22800 19500
+Wire Wire Line
+	19300 17300 17700 17300
+Wire Wire Line
+	17700 17300 17700 17650
 Wire Notes Line
 	15400 5300 13200 5300
@@
 	15250 17200 19300 17200
 Wire Wire Line
-	19300 17300 15250 17300
-Wire Wire Line
 	15250 17400 19300 17400
 Wire Wire Line
@@
 	22600 18700 22600 18550
 Wire Wire Line
-	22600 18550 23100 18550
-Wire Wire Line
-	23100 18550 23100 20100
-Wire Wire Line
-	23000 20100 23000 18650
-Wire Wire Line
-	23000 18650 22700 18650
-Wire Wire Line
 	22700 18650 22700 18700
-Wire Wire Line
-	22800 20100 22800 19500
 Wire Wire Line
 	22700 19500 22700 20100
@@
 	13900 5700 13900 6100
 Connection ~ 13900 5950
+Wire Wire Line
+	15250 17300 17250 17300
+Wire Wire Line
+	17250 17300 17250 17650
+Wire Wire Line
+	17400 17450 17400 17400
+Connection ~ 17400 17400
+Wire Wire Line
+	22800 20000 22800 20100
+Wire Wire Line
+	22600 18550 23200 18550
+Wire Wire Line
+	23200 18550 23200 20100
+$Comp
+L BUFE U?
+U 1 1 5371FE9D
+P 22800 19750
+F 0 "U?" H 23050 20200 60  0000 C CNN
+F 1 "BUFE" H 23200 20100 60  0000 C CNN
+	1    22800 19750
+	0    -1   1    0
+$EndComp
+$Comp
+L BUFE U?
+U 1 1 5371FE60
+P 17450 17650
+F 0 "U?" H 17650 17900 60  0000 C CNN
+F 1 "BUFE" H 17650 17750 60  0000 C CNN
+	1    17450 17650
+	1    0    0    1
+$EndComp
+Text Notes 13950 5800 0    90   ~ 0
+Programming mode\nbuttons
 $Comp
 L GND #PWR?
@@
 NoConn ~ 22800 18700
 Entry Wire Line
-	22900 20200 23000 20100
+	23000 20200 23100 20100
 Entry Wire Line
-	23000 20200 23100 20100
-Text Label 23000 20100 1    60   ~ 0
+	23100 20200 23200 20100
+Text Label 23100 20100 1    60   ~ 0
 MOSI
-Text Label 23100 20100 1    60   ~ 0
+Text Label 23200 20100 1    60   ~ 0
 RADIO_CSN
 $Comp
